File: connectors_pushbuttons.kicad_sch (KiCad schematic)
At the start: 28 parts, among them J1 Conn_01x12_Pin, J2 Conn_01x12_Pin, SW1 SW_Push, SW2 SW_Push, SW3 SW_Push, SW4 SW_Push, U7 74HC14, U8 74HC165

Commit message: Added 2 more pushbuttons to the 74HC165 through the Schmitt trigger inverter, removed provision for unused 74HC14 inverters as a result
Parts:
- removed R37, R38: 10k, Resistor_SMD:R_0603_1608Metric, symbol Device:R_Small
- added C1, C18: 100nF, Capacitor_SMD:C_0402_1005Metric, symbol Device:C_Small
- added R41, R42: 10k, Resistor_SMD:R_0603_1608Metric, symbol Device:R_Small
- added SW5, SW6: SW_Push, Button_Switch_SMD:SW_Push_1P1T_XKB_TS-1187A, symbol Switch:SW_Push
- renumbered R39 to R37, R40 to R38, R41 to R39, R42 to R40
Connections:
- net D2 is gone; now on net SW3: U8.13 (D2)
- net D3 is gone; now on net SW4: U8.14 (D3)
- net GPIO_B is gone; now on net SW5_PU: U7.13
- net +3V3: now also R41.1, R42.1
- net GND: now also C1.2, C18.2, SW5.1, SW6.1
- net GPIO_A renamed SW5_PU
- net SW5_PU: now also C1.1, C18.1, R41.2, R42.2, SW5.2, SW6.2
- net INV_GPIO_A renamed SW5
- net INV_GPIO_B renamed SW6
Other:
- moved on the sheet: C10, C11, C14, C15, C16, C17, R34, R35, R36, R37, R38, R39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

Commit message: Changed 100nF caps from 0402 to 0603 footprints.  Grouped all pushbuttons together and routed to PISO shift reg
Parts:
- C1, C11, C14, C15, C17, C18: footprint Capacitor_SMD:C_0402_1005Metric -> Capacitor_SMD:C_0603_1608Metric; LCSC Part # C1525 -> C14663; Manufacturer Samsung Electro-Mechanics -> YAGEO; Manufacturer Part Number CL05B104KO5NNNC -> CC0603KRX7R9BB104; Voltage (none) -> 50V
Connections:
- net SW5_PU: no longer C18.1, R42.2, SW6.2, U7.13
- net BUTTON_CE: now reaches R43.1, U8.15 (~{CE})
- new net SW6_PU: C18.1, R42.2, SW6.2, U7.13
